Commit message: arm added

File: src/titan_description/urdf/macros.xacro (robot description, xacro)
@@ -13,3 +13,33 @@
 		<inertia  ixx="${m*(3*r*r+h*h)/12}" ixy = "0" ixz = "0" iyy="${m*(3*r*r+h*h)/12}" iyz = "0" izz="${m*r*r/2}"/>
 	</xacro:macro>
+	<xacro:macro name="make_box" params="x y z roll pitch yaw sizex sizey sizez">
+		<collision name='collision'>
+			<origin xyz="${x} ${y} ${z}" rpy="${roll} ${pitch} ${yaw}"/>
+			<geometry>
+				<box size="${sizex} ${sizey} ${sizez}"/>
+			</geometry>
+		</collision>
+		<visual name='visual'>
+			<origin xyz="${x} ${y} ${z}" rpy="${roll} ${pitch} ${yaw}"/>
+			<geometry>
+				<box size="${sizex} ${sizey} ${sizez}"/>
+			</geometry>
+			<material name="white"/>
+		</visual>
+	</xacro:macro>
+        <!-- <xacro:macro name="make_cylinder" params="x y z roll pitch yaw r h">
+		<collision name='collision'>
+			<origin xyz="${x} ${y} ${z}" rpy="${roll} ${pitch} ${yaw}"/>
+			<geometry>
+				 <cylinder length="${r}" length="${h}"/>
+			</geometry>
+		</collision>
+		<visual name='visual'>
+			<origin xyz="${x} ${y} ${z}" rpy="${roll} ${pitch} ${yaw}"/>
+			<geometry>
+				<cylinder length="${r}" length="${h}"/>
+			</geometry>
+			<material name="white"/>
+		</visual>
+        </xacro:macro> -->
 </robot>

Commit message: updates

File: src/titan_description/urdf/macros.xacro (robot description, xacro)
@@ -1,4 +1,4 @@
 <?xml version='1.0'?>
-<robot name="titan" xmlns:xacro="http://www.ros.org/wiki/xacro">
+<robot name="titan" xmlns:xacro="http://ros.org/wiki/xacro">
 	<xacro:macro name="default_inertial" params="mass">
 		<inertial>

File: src/titan_description/urdf/titan.xacro (robot description, xacro)
@@ -1,4 +1,4 @@
 <?xml version='1.0'?>
-<robot name="titan" xmlns:xacro="http://www.ros.org/wiki/xacro">
+<robot name="titan" xmlns:xacro="http://ros.org/wiki/xacro">
 	<xacro:property name="M_PI" value="3.14159"/>
 	<xacro:property name="rotate90CCW" value="${3.14159 / 2}"/>
@@ -106,6 +106,5 @@
 		<parent link="base_link"/>
 		<child link="laser_mount_link"/>
-		<!-- <origin xyz="0.025 0.08 ${(base_z_size/2) + plate_offset + laser_z_size}" rpy="0 0 0" /> -->
-		<origin xyz="0.0 0.0 ${(base_z_size/2) + plate_offset + 0.05}" rpy="0 0 0" />
+		<origin xyz="0.193 0.035 ${(base_z_size/2) + plate_offset + 0.05}" rpy="0 0 0" />
 	</joint>
 	<joint name="base_to_imu_link" type="fixed">

File: src/titan_description/urdf/wheel.xacro (robot description, xacro)
@@ -1,3 +1,3 @@
-<robot xmlns:xacro="http://www.ros.org/wiki/xacro" name="titan_wheel">
+<robot xmlns:xacro="http://ros.org/wiki/xacro" name="titan_wheel">
 	<xacro:macro name="titan_wheel" params="wheel_prefix *joint_pose">
 		<link name="${wheel_prefix}_wheel_link">
