Commit message: action server and traj working

File: src/titan_description/urdf/arm.xacro (robot description, xacro)
@@ -81,5 +81,5 @@
 		<parent link="link3"/>
 		<child link="end_effector"/>
-                <origin xyz="${link3_base_x_size} 0 ${-eef_z_size/2}" rpy="0 0 0"/>
+                <origin xyz="${link3_base_x_size} 0 ${-eef_z_size + 0.001}" rpy="0 0 0"/>
 	</joint>
 </robot>

File: src/titan_description/urdf/titan.xacro (robot description, xacro)
@@ -25,13 +25,10 @@
 	<xacro:property name="short_channel_y" value="0.0381"/>
 	<xacro:property name="short_channel_mass" value="0.0952544"/>
-	<xacro:property name="wheelbase" value="0.23" />
+	<xacro:property name="wheelbase" value="0.345" />
 	<xacro:property name="track" value="0.355" />
-	<!-- <xacro:property name="wheelbase" value="1.0" />
-	<xacro:property name="track" value="1.0" /> -->
-	<xacro:property name="wheel_vertical_offset" value="0.06" />
-	<xacro:property name="wheel_length" value="0.025" />
-	<xacro:property name="wheel_radius" value="0.0508" />
-	<!-- <xacro:property name="wheel_radius" value="1.0" /> -->
-	<xacro:property name="camera_link" value="0.05" /> <!-- Size of square 'camera' box -->
+	<xacro:property name="wheel_vertical_offset" value="0.0762" />
+	<xacro:property name="wheel_radius" value="0.0762" />
+	<xacro:property name="wheel_length" value="${wheel_radius*2}" />
+	<xacro:property name="camera_link" value="0.05" />
 	<xacro:arg name="robot_namespace" default="/" />
 	<xacro:include filename="$(find titan_description)/urdf/materials.xacro" />

Commit message: updates

File: src/titan_description/urdf/arm.xacro (robot description, xacro)
@@ -67,5 +67,5 @@
 		<parent link="link1"/>
 		<child link="link2"/>
-		<limit effort="1000.0" lower="-2" upper="2" velocity="0.5"/>
+		<limit effort="1000.0" lower="-2" upper="2" velocity="0.45"/>
 		<axis xyz="0 0 1"/>
 		<origin xyz="${link1_base_z_size/2} 0 ${-link1_base_z_size}" rpy="0 0 0" />
@@ -74,10 +74,12 @@
 		<parent link="link2"/>
 		<child link="link3"/>
-		<limit effort="1000.0" lower="-3.0" upper="3.0" velocity="0.5"/>
+		<limit effort="1000.0" lower="-3.0" upper="3.0" velocity="0.255"/>
 		<axis xyz="0 0 1"/>
 		<origin xyz="${link2_base_x_size} 0 ${-link2_base_z_size}" rpy="0 0 0" />
 	</joint>
-	<joint name="link3_to_eef" type="fixed">
+	<joint name="link3_to_eef" type="revolute">
 		<parent link="link3"/>
+		<limit effort="1000.0" lower="${-1.57}" upper="1.57" velocity="0.35"/>
+		<axis xyz="0 0 1"/>
 		<child link="end_effector"/>
                 <origin xyz="${link3_base_x_size} 0 ${-eef_z_size + 0.001}" rpy="0 0 0"/>

Commit message: arm update

File: src/titan_description/urdf/arm.xacro (robot description, xacro)
@@ -55,5 +55,5 @@
 		<parent link="arm_base_link"/>
 		<child link="zaxis_base_link"/>
-		<limit effort="1000.0" lower="0.0" upper="${arm_base_z_size - zaxis_base_z_size}" velocity="0.5"/>
+		<limit effort="1000.0" lower="0.0" upper="${arm_base_z_size }" velocity="0.5"/>
 		<axis xyz="0 0 1"/>
 		<origin xyz="0.05 0 ${-arm_base_z_size/2 + zaxis_base_z_size/2}"/>
