Commit message: merge arm and base

File: src/titan_description/urdf/titan_base.xacro (robot description, xacro)
@@ -18,28 +18,4 @@
 	<xacro:property name="wheel_radius" value="0.09" />
 	<xacro:property name="wheel_length" value="0.0508" />
-	<xacro:property name="arm_base_x_size" value="0.0381"/>
-	<xacro:property name="arm_base_y_size" value="0.1143"/>
-	<xacro:property name="arm_base_z_size" value="0.6096"/>
-	<xacro:property name="arm_base_mass" value="0.3"/>
-	<xacro:property name="zaxis_base_x_size" value="0.0381"/>
-	<xacro:property name="zaxis_base_y_size" value="0.1143"/>
-	<xacro:property name="zaxis_base_z_size" value="0.1524"/>
-	<xacro:property name="zaxis_base_mass" value="0.05"/>
-	<xacro:property name="link1_base_x_size" value="0.09"/>
-	<xacro:property name="link1_base_y_size" value="0.0381"/>
-	<xacro:property name="link1_base_z_size" value="0.0381"/>
-	<xacro:property name="link1_base_mass" value="0.05"/>
-	<xacro:property name="link2_base_x_size" value="0.5"/>
-	<xacro:property name="link2_base_y_size" value="0.0381"/>
-	<xacro:property name="link2_base_z_size" value="0.0381"/>
-	<xacro:property name="link2_base_mass" value="0.05"/>
-	<xacro:property name="link3_base_x_size" value="0.5"/>
-	<xacro:property name="link3_base_y_size" value="0.0381"/>
-	<xacro:property name="link3_base_z_size" value="0.0381"/>
-	<xacro:property name="link3_base_mass" value="0.05"/>
-	<xacro:property name="eef_x_size" value="0.0381"/>
-	<xacro:property name="eef_y_size" value="0.0381"/>
-	<xacro:property name="eef_z_size" value="0.15"/>
-	<xacro:property name="eef_mass" value="0.05"/>
 	<xacro:property name="camera_link" value="0.05" />
 	<xacro:arg name="robot_namespace" default="/" />
@@ -103,24 +79,4 @@
                 </inertial> -->
         </link>
-	<link name="arm_base_link">
-		<pose xyz="0 0 0" rpy="0 0 0" />
-		<xacro:box_inertia m="${arm_base_mass}" x="${arm_base_x_size}" y="${arm_base_y_size}" z="${arm_base_z_size}" />
-		<xacro:make_box x="0" y="0" z="0" roll="0" pitch="0" yaw="0" sizex="${arm_base_x_size}" sizey="${arm_base_y_size}" sizez="${arm_base_z_size}"/>
-	</link>
-	<link name="zaxis_base_link">
-		<xacro:make_box x="0" y="0" z="0" roll="0" pitch="0" yaw="0" sizex="${zaxis_base_x_size}" sizey="${zaxis_base_y_size}" sizez="${zaxis_base_z_size}"/>
-	</link>
-	<link name="link1">
-		<xacro:make_box x="0" y="0" z="0" roll="0" pitch="0" yaw="0" sizex="${link1_base_x_size}" sizey="${link1_base_y_size}" sizez="${link1_base_z_size}"/>
-	</link>
-	<link name="link2">
-		<xacro:make_box x="${link2_base_x_size/2}" y="0" z="0" roll="0" pitch="0" yaw="0" sizex="${link2_base_x_size}" sizey="${link2_base_y_size}" sizez="${link2_base_z_size}"/>
-	</link>
-	<link name="link3">
-		<xacro:make_box x="${link3_base_x_size/2}" y="0" z="0" roll="0" pitch="0" yaw="0" sizex="${link3_base_x_size}" sizey="${link3_base_y_size}" sizez="${link3_base_z_size}"/>
-	</link>
-	<link name="end_effector">
-		<xacro:make_box x="0" y="0" z="0" roll="0" pitch="0" yaw="0" sizex="${eef_x_size}" sizey="${eef_y_size}" sizez="${eef_z_size}"/>
-	</link>
 	<joint name="base_to_inertia" type="fixed">
 		<parent link="base_link"/>
@@ -142,42 +98,4 @@
 		<child link="imu_link"/>
 		<origin xyz="0 0 ${(base_z_size/2)  + 0.02}" rpy="0 0 0"/>
-	</joint>
-	<joint name="base_to_arm" type="fixed">
-		<parent link="base_link"/>
-		<child link="arm_base_link"/>
-		<origin xyz="0.0 -0.13 ${arm_base_z_size/2}"/>
-	</joint>
-	<joint name="base_to_zaxis" type="prismatic">
-		<parent link="arm_base_link"/>
-		<child link="zaxis_base_link"/>
-		<limit effort="1000.0" lower="0.0" upper="${arm_base_z_size }" velocity="0.5"/>
-		<axis xyz="0 0 -1"/>
-		<origin xyz="0.05 0 ${arm_base_z_size/2 - zaxis_base_z_size/2}"/>
-	</joint>
-	<joint name="zaxis_to_link1" type="fixed">
-		<parent link="zaxis_base_link"/>
-		<child link="link1"/>
-		<origin xyz="${zaxis_base_x_size/2 + link1_base_x_size/2} 0 0" rpy="0 0 0"/>
-	</joint>
-	<joint name="link1_to_link2" type="revolute">
-		<parent link="link1"/>
-		<child link="link2"/>
-		<limit effort="1000.0" lower="-2" upper="2" velocity="0.45"/>
-		<axis xyz="0 0 1"/>
-		<origin xyz="${link1_base_z_size/2} 0 ${-link1_base_z_size}" rpy="0 0 0" />
-	</joint>
-	<joint name="link2_to_link3" type="revolute">
-		<parent link="link2"/>
-		<child link="link3"/>
-		<limit effort="1000.0" lower="-3.0" upper="3.0" velocity="0.255"/>
-		<axis xyz="0 0 1"/>
-		<origin xyz="${link2_base_x_size} 0 ${-link2_base_z_size}" rpy="0 0 0" />
-	</joint>
-	<joint name="link3_to_eef" type="revolute">
-		<parent link="link3"/>
-		<limit effort="1000.0" lower="${-1.57}" upper="1.57" velocity="0.35"/>
-		<axis xyz="0 0 1"/>
-		<child link="end_effector"/>
-                <origin xyz="${link3_base_x_size} 0 ${-eef_z_size + 0.001}" rpy="0 0 0"/>
 	</joint>
 	<xacro:titan_wheel wheel_prefix="left_front">
