Commit message: nav updates

File: src/titan_description/urdf/titan.xacro (robot description, xacro)
@@ -102,5 +102,5 @@
 		<parent link="base_link"/>
 		<child link="laserbox_link"/>
-		<origin xyz="0.16 0 ${(base_z_size/2) + plate_offset + laser_z_size}"/>
+		<origin xyz="0.16 0 ${(base_z_size/2) + plate_offset + laser_z_size}" rpy="0 0 3.14" />
 	</joint>
 	<joint name="laserbox_to_laser" type="fixed">

Commit message: Sensor fusion working

File: src/titan_description/urdf/titan.xacro (robot description, xacro)
@@ -25,6 +25,6 @@
 	<xacro:property name="short_channel_y" value="0.0381"/>
 	<xacro:property name="short_channel_mass" value="0.0952544"/>
-	<xacro:property name="wheelbase" value="0.2" />
-	<xacro:property name="track" value="0.345" />
+	<xacro:property name="wheelbase" value="0.23" />
+	<xacro:property name="track" value="0.355" />
 	<!-- <xacro:property name="wheelbase" value="1.0" />
 	<xacro:property name="track" value="1.0" /> -->
@@ -112,5 +112,5 @@
 		<parent link="base_link"/>
 		<child link="imu_link"/>
-		<origin xyz="0.16 0 ${(base_z_size/2) + plate_offset + 0.02}"/>
+		<origin xyz="0.16 0 ${(base_z_size/2) + plate_offset + 0.02}" rpy="0 0 ${3.14}"/>
 	</joint>
 	<xacro:titan_wheel wheel_prefix="front_left">

Commit message: fixed wheel urdf

File: src/titan_description/urdf/titan.xacro (robot description, xacro)
@@ -29,5 +29,5 @@
 	<xacro:property name="wheel_vertical_offset" value="0.0762" />
 	<xacro:property name="wheel_radius" value="0.0762" />
-	<xacro:property name="wheel_length" value="${wheel_radius*2}" />
+	<xacro:property name="wheel_length" value="0.025" />
 	<xacro:property name="camera_link" value="0.05" />
 	<xacro:arg name="robot_namespace" default="/" />

Commit message: new frame layout fixes

File: src/titan_description/urdf/titan.xacro (robot description, xacro)
@@ -91,4 +91,13 @@
 		</visual>
 	</link>
+	<link name="camera_link">
+                <visual name='camera_box'>
+                        <origin xyz="0 0 0" rpy="0 0 0"/>
+                        <geometry>
+                                <box size="0.05 0.05 0.05"/>
+                        </geometry>
+                        <material name="green"/>
+                </visual>
+        </link>
 	<joint name="base_to_inertia" type="fixed">
 		<parent link="base_link"/>
@@ -96,8 +105,13 @@
 		<origin xyz="0 0 0"/>
 	</joint>
+	<joint name="base_to_camera" type="fixed">
+                <parent link="base_link"/>
+                <child link="camera_link"/>
+                <origin xyz="0.2 0 ${(base_z_size/2) + plate_offset + 0.05}" rpy="0 0 0" />
+        </joint>
 	<joint name="base_to_laserbox" type="fixed">
 		<parent link="base_link"/>
 		<child link="laserbox_link"/>
-		<origin xyz="0.16 0 ${(base_z_size/2) + plate_offset + laser_z_size}" rpy="0 0 3.14" />
+		<origin xyz="0.025 0.08 ${(base_z_size/2) + plate_offset + laser_z_size}" rpy="0 0 0" />
 	</joint>
 	<joint name="laserbox_to_laser" type="fixed">
@@ -109,5 +123,5 @@
 		<parent link="base_link"/>
 		<child link="imu_link"/>
-		<origin xyz="0.16 0 ${(base_z_size/2) + plate_offset + 0.02}" rpy="0 0 ${3.14}"/>
+		<origin xyz="-0.050 -0.010 ${(base_z_size/2) + plate_offset + 0.02}" rpy="0 0 ${0}"/>
 	</joint>
 	<xacro:titan_wheel wheel_prefix="front_left">

Commit message: Updates

File: src/titan_description/urdf/titan.xacro (robot description, xacro)
@@ -73,5 +73,5 @@
 		</visual>
 	</link>
-	<link name="laser_link">
+	<link name="laser">
 		<visual name='laser'>
 			<origin xyz="0 0 0" rpy="0 0 0"/>
@@ -117,5 +117,5 @@
 	<joint name="laserbox_to_laser" type="fixed">
 		<parent link="laserbox_link"/>
-		<child link="laser_link"/>
+		<child link="laser"/>
 		<origin xyz="0 0 ${(laser_z_size/2)+ (0.01/2)}"/>
 	</joint>

Commit message: updates

File: src/titan_description/urdf/titan.xacro (robot description, xacro)
@@ -82,5 +82,5 @@
 		</visual>
 	</link>
-	<link name="imu_link">
+	<!-- <link name="imu_link">
 		<visual name='imu_box'>
 			<origin xyz="0 0 0" rpy="0 0 0"/>
@@ -90,5 +90,5 @@
 			<material name="green"/>
 		</visual>
-	</link>
+	</link> -->
 	<link name="camera_link">
                 <visual name='camera_box'>
@@ -108,10 +108,11 @@
                 <parent link="base_link"/>
                 <child link="camera_link"/>
-                <origin xyz="0.2 0 ${(base_z_size/2) + plate_offset + 0.05}" rpy="0 0 0" />
+                <origin xyz="0.0 0 ${(base_z_size/2) + plate_offset + 0.3}" rpy="0 0 0" />
         </joint>
 	<joint name="base_to_laserbox" type="fixed">
 		<parent link="base_link"/>
 		<child link="laserbox_link"/>
-		<origin xyz="0.025 0.08 ${(base_z_size/2) + plate_offset + laser_z_size}" rpy="0 0 0" />
+		<!-- <origin xyz="0.025 0.08 ${(base_z_size/2) + plate_offset + laser_z_size}" rpy="0 0 0" /> -->
+		<origin xyz="0.2 0 ${(base_z_size/2) + plate_offset + 0.05}" rpy="0 0 0" />
 	</joint>
 	<joint name="laserbox_to_laser" type="fixed">
@@ -120,9 +121,9 @@
 		<origin xyz="0 0 ${(laser_z_size/2)+ (0.01/2)}"/>
 	</joint>
-	<joint name="base_to_imu_link" type="fixed">
+	<!-- <joint name="base_to_imu_link" type="fixed">
 		<parent link="base_link"/>
 		<child link="imu_link"/>
 		<origin xyz="-0.050 -0.010 ${(base_z_size/2) + plate_offset + 0.02}" rpy="0 0 ${0}"/>
-	</joint>
+	</joint> -->
 	<xacro:titan_wheel wheel_prefix="front_left">
 		<origin xyz="${wheelbase/2} ${track/2} ${wheel_vertical_offset}" rpy="0 0 0" />

Commit message: updates

File: src/titan_description/urdf/titan.xacro (robot description, xacro)
@@ -124,5 +124,5 @@
 		<parent link="base_link"/>
 		<child link="imu_link"/>
-		<origin xyz="-0.050 -0.010 ${(base_z_size/2) + plate_offset + 0.02}" rpy="0 0 ${0}"/>
+		<origin xyz="0 0 ${(base_z_size/2) + plate_offset + 0.02}" rpy="0 0 0"/>
 	</joint> -->
 	<xacro:titan_wheel wheel_prefix="front_left">

Commit message: stuffs

File: src/titan_description/urdf/titan.xacro (robot description, xacro)
@@ -37,5 +37,5 @@
 	<xacro:include filename="$(find titan_description)/urdf/titan.gazebo" />
 	<link name="base_link">
-		<pose xyz="0 0 1" rpy="0 0 0" />
+		<pose xyz="0 0 0" rpy="0 0 0" />
 		<!-- <inertial>
 			<mass value="${total_mass}" />
@@ -82,5 +82,5 @@
 		</visual>
 	</link>
-	<!-- <link name="imu_link">
+	<link name="imu_link">
 		<visual name='imu_box'>
 			<origin xyz="0 0 0" rpy="0 0 0"/>
@@ -90,5 +90,5 @@
 			<material name="green"/>
 		</visual>
-	</link> -->
+	</link>
 	<link name="camera_link">
                 <visual name='camera_box'>
@@ -121,9 +121,9 @@
 		<origin xyz="0 0 ${(laser_z_size/2)+ (0.01/2)}"/>
 	</joint>
-	<!-- <joint name="base_to_imu_link" type="fixed">
+	<joint name="base_to_imu_link" type="fixed">
 		<parent link="base_link"/>
 		<child link="imu_link"/>
 		<origin xyz="0 0 ${(base_z_size/2) + plate_offset + 0.02}" rpy="0 0 0"/>
-	</joint> -->
+	</joint>
 	<xacro:titan_wheel wheel_prefix="front_left">
 		<origin xyz="${wheelbase/2} ${track/2} ${wheel_vertical_offset}" rpy="0 0 0" />

Commit message: updates

File: src/titan_description/urdf/titan.xacro (robot description, xacro)
@@ -36,4 +36,5 @@
 	<xacro:include filename="$(find titan_description)/urdf/wheel.xacro" />
 	<xacro:include filename="$(find titan_description)/urdf/titan.gazebo" />
+	<xacro:include filename="$(find titan_description)/urdf/sick_tim.urdf.xacro" />
 	<link name="base_link">
 		<pose xyz="0 0 0" rpy="0 0 0" />
@@ -64,14 +65,5 @@
 		</inertial>
 	</link>
-	<link name="laserbox_link">
-		<visual name='laser_box'>
-			<origin xyz="0 0 0" rpy="0 0 0"/>
-			<geometry>
-				<box size="${laser_x_size} ${laser_y_size} ${laser_z_size}"/>
-			</geometry>
-			<material name="black"/>
-		</visual>
-	</link>
-	<link name="laser">
+	<!-- <link name="laser">
 		<visual name='laser'>
 			<origin xyz="0 0 0" rpy="0 0 0"/>
@@ -81,5 +73,6 @@
 			<material name="red"/>
 		</visual>
-	</link>
+	</link> -->
+	<xacro:sick_tim551 name="laser" ros_topic="scan" />
 	<link name="imu_link">
 		<visual name='imu_box'>
@@ -110,14 +103,9 @@
                 <origin xyz="0.0 0 ${(base_z_size/2) + plate_offset + 0.3}" rpy="0 0 0" />
         </joint>
-	<joint name="base_to_laserbox" type="fixed">
+	<joint name="base_to_laser" type="fixed">
 		<parent link="base_link"/>
-		<child link="laserbox_link"/>
+		<child link="laser_mount_link"/>
 		<!-- <origin xyz="0.025 0.08 ${(base_z_size/2) + plate_offset + laser_z_size}" rpy="0 0 0" /> -->
-		<origin xyz="0.2 0 ${(base_z_size/2) + plate_offset + 0.05}" rpy="0 0 0" />
-	</joint>
-	<joint name="laserbox_to_laser" type="fixed">
-		<parent link="laserbox_link"/>
-		<child link="laser"/>
-		<origin xyz="0 0 ${(laser_z_size/2)+ (0.01/2)}"/>
+		<origin xyz="0.0 0.0 ${(base_z_size/2) + plate_offset + 0.05}" rpy="0 0 0" />
 	</joint>
 	<joint name="base_to_imu_link" type="fixed">

Commit message: camera urdf

File: src/titan_description/urdf/titan.xacro (robot description, xacro)
@@ -101,5 +101,5 @@
                 <parent link="base_link"/>
                 <child link="camera_link"/>
-                <origin xyz="0.0 0 ${(base_z_size/2) + plate_offset + 0.3}" rpy="0 0 0" />
+                <origin xyz="0.13 0.08 ${(base_z_size/2) + plate_offset + 0.3}" rpy="0 0 0" />
         </joint>
 	<joint name="base_to_laser" type="fixed">

Commit message: description updates

File: src/titan_description/urdf/titan.xacro (robot description, xacro)
@@ -5,29 +5,17 @@
 	<xacro:property name="rotate90CW" value="${-3.14159 / 2}"/>
 	<xacro:property name="total_mass" value="15"/>
-	<xacro:property name="plate_x" value="0.2286"/>
-	<xacro:property name="plate_y" value="0.3048"/>
-	<xacro:property name="plate_z" value="0.002286"/>
-	<xacro:property name="plate_offset" value="0.0508"/>
-	<xacro:property name="plate_mass" value="0.317515"/>
-	<xacro:property name="base_x_size" value="${plate_x*2}"/>
-	<xacro:property name="base_y_size" value="${plate_y}"/>
-	<xacro:property name="base_z_size" value="0.075"/>
-	<xacro:property name="base_mass" value="${plate_mass*2}"/>
+	<xacro:property name="base_x_size" value="0.7556"/>
+	<xacro:property name="base_y_size" value="0.4572"/>
+	<xacro:property name="base_z_size" value="0.0508"/>
+	<xacro:property name="base_mass" value="10"/>
 	<xacro:property name="laser_x_size" value="0.125"/>
 	<xacro:property name="laser_y_size" value="0.105"/>
 	<xacro:property name="laser_z_size" value="0.07"/>
 	<xacro:property name="laser_mass" value="0.05"/>
-	<xacro:property name="long_channel_x" value="0.4572"/>
-	<xacro:property name="long_channel_y" value="0.0381"/>
-	<xacro:property name="long_channel_z" value="0.002286"/>
-	<xacro:property name="long_channel_mass" value="0.1950447"/>
-	<xacro:property name="short_channel_x" value="0.4572"/>
-	<xacro:property name="short_channel_y" value="0.0381"/>
-	<xacro:property name="short_channel_mass" value="0.0952544"/>
-	<xacro:property name="wheelbase" value="0.345" />
-	<xacro:property name="track" value="0.355" />
-	<xacro:property name="wheel_vertical_offset" value="0.0762" />
-	<xacro:property name="wheel_radius" value="0.0762" />
-	<xacro:property name="wheel_length" value="0.025" />
+	<xacro:property name="wheelbase" value="0.58" />
+	<xacro:property name="track" value="0.25" />
+	<xacro:property name="wheel_vertical_offset" value="0.0" />
+	<xacro:property name="wheel_radius" value="0.097155" />
+	<xacro:property name="wheel_length" value="0.0508" />
 	<xacro:property name="camera_link" value="0.05" />
 	<xacro:arg name="robot_namespace" default="/" />
@@ -39,11 +27,6 @@
 	<link name="base_link">
 		<pose xyz="0 0 0" rpy="0 0 0" />
-		<!-- <inertial>
-			<mass value="${total_mass}" />
-			<origin xyz="0 0 ${(base_z_size/2) + plate_offset}" rpy=" 0 0 0"/>
-			<xacro:box_inertia m="${total_mass}" x="${base_x_size}" y="${base_y_size}" z="${base_z_size}" />
-		</inertial> -->
 		<collision name='collision'>
-			<origin xyz="0 0 ${(base_z_size/2) + plate_offset}" rpy="0 0 0" />
+			<origin xyz="0 0 ${-(base_z_size/2)}" rpy="0 0 0" />
 			<geometry>
 				<box size="${base_x_size} ${base_y_size} ${base_z_size}"/>
@@ -51,5 +34,5 @@
 		</collision>
 		<visual name='base_solid'>
-			<origin xyz="0 0 ${(base_z_size/2) + plate_offset}" rpy="0 0 0" />
+			<origin xyz="0 0 ${-(base_z_size/2)}" rpy="0 0 0" />
 			<geometry>
 				<box size="${base_x_size} ${base_y_size} ${base_z_size}"/>
@@ -61,17 +44,8 @@
 		<inertial>
 			<mass value="${total_mass}" />
-			<origin xyz="0 0 ${(base_z_size/2) + plate_offset}" rpy=" 0 0 0"/>
+			<origin xyz="0 0 0" rpy=" 0 0 0"/>
 			<xacro:box_inertia m="${total_mass}" x="${base_x_size}" y="${base_y_size}" z="${base_z_size}" />
 		</inertial>
 	</link>
-	<!-- <link name="laser">
-		<visual name='laser'>
-			<origin xyz="0 0 0" rpy="0 0 0"/>
-			<geometry>
-				<cylinder length="0.01" radius="0.04"/>
-			</geometry>
-			<material name="red"/>
-		</visual>
-	</link> -->
 	<xacro:sick_tim551 name="laser" ros_topic="scan" />
 	<link name="imu_link">
@@ -101,27 +75,33 @@
                 <parent link="base_link"/>
                 <child link="camera_link"/>
-                <origin xyz="0.13 0.08 ${(base_z_size/2) + plate_offset + 0.3}" rpy="0 0 0" />
+                <origin xyz="0.13 0.08 ${(base_z_size/2) + 0.3}" rpy="0 0 0" />
         </joint>
 	<joint name="base_to_laser" type="fixed">
 		<parent link="base_link"/>
 		<child link="laser_mount_link"/>
-		<origin xyz="0.193 0.035 ${(base_z_size/2) + plate_offset + 0.05}" rpy="0 0 0" />
+		<origin xyz="0.31 0.0 0.08" rpy="0 0 0" />
 	</joint>
 	<joint name="base_to_imu_link" type="fixed">
 		<parent link="base_link"/>
 		<child link="imu_link"/>
-		<origin xyz="0 0 ${(base_z_size/2) + plate_offset + 0.02}" rpy="0 0 0"/>
+		<origin xyz="0 0 ${(base_z_size/2)  + 0.02}" rpy="0 0 0"/>
 	</joint>
-	<xacro:titan_wheel wheel_prefix="front_left">
-		<origin xyz="${wheelbase/2} ${track/2} ${wheel_vertical_offset}" rpy="0 0 0" />
+	<xacro:titan_wheel wheel_prefix="left_front">
+		<origin xyz="${track} ${wheelbase/2} ${wheel_vertical_offset}" rpy="0 0 0" />
 	</xacro:titan_wheel>
-	<xacro:titan_wheel wheel_prefix="front_right">
-		<origin xyz="${wheelbase/2} ${-track/2} ${wheel_vertical_offset}" rpy="0 0 0" />
+	<xacro:titan_wheel wheel_prefix="left_mid">
+                <origin xyz="0 ${wheelbase/2} ${wheel_vertical_offset}" rpy="0 0 0" />
+        </xacro:titan_wheel>
+	<xacro:titan_wheel wheel_prefix="left_rear">
+		<origin xyz="${-track} ${wheelbase/2} ${wheel_vertical_offset}" rpy="0 0 0" />
 	</xacro:titan_wheel>
-	<xacro:titan_wheel wheel_prefix="rear_left">
-		<origin xyz="${-wheelbase/2} ${track/2} ${wheel_vertical_offset}" rpy="0 0 0" />
+	<xacro:titan_wheel wheel_prefix="right_front">
+		<origin xyz="${track} ${-wheelbase/2} ${wheel_vertical_offset}" rpy="0 0 0" />
 	</xacro:titan_wheel>
-	<xacro:titan_wheel wheel_prefix="rear_right">
-	<origin xyz="${-wheelbase/2} ${-track/2} ${wheel_vertical_offset}" rpy="0 0 0" />
+	<xacro:titan_wheel wheel_prefix="right_mid">
+                <origin xyz="0 ${-wheelbase/2} ${wheel_vertical_offset}" rpy="0 0 0" />
+        </xacro:titan_wheel>
+	<xacro:titan_wheel wheel_prefix="right_rear">
+		<origin xyz="${-track} ${-wheelbase/2} ${wheel_vertical_offset}" rpy="0 0 0" />
 	</xacro:titan_wheel>
 	<gazebo>

Commit message: updates

File: src/titan_description/urdf/titan.xacro (robot description, xacro)
@@ -16,5 +16,5 @@
 	<xacro:property name="track" value="0.25" />
 	<xacro:property name="wheel_vertical_offset" value="0.0" />
-	<xacro:property name="wheel_radius" value="0.097155" />
+	<xacro:property name="wheel_radius" value="0.09" />
 	<xacro:property name="wheel_length" value="0.0508" />
 	<xacro:property name="camera_link" value="0.05" />

Commit message: updates for gazebo

File: src/titan_description/urdf/titan.xacro (robot description, xacro)
@@ -58,4 +58,6 @@
 		</visual>
 	</link>
+	<gazebo reference="imu_link">
+  	</gazebo>
 	<link name="camera_link">
                 <visual name='camera_box'>
@@ -110,5 +112,5 @@
 		</plugin>
 	</gazebo>
-	<gazebo>
+	<!--<gazebo>
 		<plugin name="skid_steer_drive_controller" filename="libgazebo_ros_skid_steer_drive.so">
 			<updateRate>100.0</updateRate>
@@ -127,4 +129,18 @@
 			<broadcastTF>false</broadcastTF>
 		</plugin>
+	</gazebo> -->
+	<gazebo>
+		<plugin name="imu_controller" filename="libhector_gazebo_ros_imu.so">
+			<robotNamespace>$(arg robot_namespace)</robotNamespace>
+			<updateRate>50.0</updateRate>
+			<bodyName>base_link</bodyName>
+			<topicName>imu/data</topicName>
+			<accelDrift>0.005 0.005 0.005</accelDrift>
+			<accelGaussianNoise>0.005 0.005 0.005</accelGaussianNoise>
+			<rateDrift>0.005 0.005 0.005 </rateDrift>
+			<rateGaussianNoise>0.005 0.005 0.005 </rateGaussianNoise>
+			<headingDrift>0.005</headingDrift>
+			<headingGaussianNoise>0.005</headingGaussianNoise>
+		</plugin>
 	</gazebo>
 </robot>

File: src/titan_description/urdf/wheel.xacro (robot description, xacro)
@@ -22,11 +22,10 @@
 		</link>
 		<gazebo reference="${wheel_prefix}_wheel_link">
-			<mu1 value="10000.0" />
-			<mu2 value="10000.0" />
-			<kp value="100000.0" />
-			<kd value="0.00001" />
+			<mu1 value="1.0" />
+			<mu2 value="1.0" />
+			<kp value="10000000.0" />
+			<kd value="1.0" />
 			<maxVel value="1.0" />
-			<minDepth value="0.0001" />
-			<fdir1 value="0 1 0"/>
+			<fdir1 value="1 0 0"/>
 		</gazebo>
 		<joint name="${wheel_prefix}_wheel" type="continuous">
@@ -35,6 +34,5 @@
 			<xacro:insert_block name="joint_pose"/>
 			<axis xyz="0 1 0" rpy="0 0 0" />
-			<limit effort="10000" velocity="1000"/>
-			<joint_properties damping="0.0" friction="0.0"/>
+			<!-- <joint_properties damping="0.0" friction="0.0"/> -->
 		</joint>
 		<transmission name="${wheel_prefix}_wheel_trans" type="SimpleTransmission">
@@ -44,5 +42,5 @@
 			</actuator>
 			<joint name="${wheel_prefix}_wheel">
-				<hardwareInterface>EffortJointInterface</hardwareInterface>
+				<hardwareInterface>hardware_interface/VelocityJointInterface</hardwareInterface>
 			</joint>
 		</transmission>

Commit message: updates

File: src/titan_description/urdf/titan.xacro (robot description, xacro)
@@ -57,4 +57,9 @@
 			<material name="green"/>
 		</visual>
+		<inertial>
+                        <mass value="${0.005}" />
+                        <origin xyz="0 0 0" rpy=" 0 0 0"/>
+                        <xacro:box_inertia m="${0.005}" x="${0.05}" y="${0.05}" z="${0.05}" />
+                </inertial>
 	</link>
 	<gazebo reference="imu_link">
@@ -68,4 +73,9 @@
                         <material name="green"/>
                 </visual>
+		<inertial>
+                        <mass value="${0.05}" />
+                        <origin xyz="0 0 0" rpy=" 0 0 0"/>
+                        <xacro:box_inertia m="${0.005}" x="${0.05}" y="${0.05}" z="${0.05}" />
+                </inertial>
         </link>
 	<joint name="base_to_inertia" type="fixed">

Commit message: gazebo updates

File: src/titan_description/urdf/titan.xacro (robot description, xacro)
@@ -57,9 +57,9 @@
 			<material name="green"/>
 		</visual>
-		<inertial>
+		<!-- <inertial>
                         <mass value="${0.005}" />
                         <origin xyz="0 0 0" rpy=" 0 0 0"/>
                         <xacro:box_inertia m="${0.005}" x="${0.05}" y="${0.05}" z="${0.05}" />
-                </inertial>
+                </inertial> -->
 	</link>
 	<gazebo reference="imu_link">
@@ -73,9 +73,9 @@
                         <material name="green"/>
                 </visual>
-		<inertial>
+		<!-- <inertial>
                         <mass value="${0.05}" />
                         <origin xyz="0 0 0" rpy=" 0 0 0"/>
                         <xacro:box_inertia m="${0.005}" x="${0.05}" y="${0.05}" z="${0.05}" />
-                </inertial>
+                </inertial> -->
         </link>
 	<joint name="base_to_inertia" type="fixed">
@@ -141,4 +141,28 @@
 	</gazebo> -->
 	<gazebo>
+		<plugin name="differential_drive_controller" filename="libgazebo_ros_diff_drive.so">
+		<robotNamespace>$(arg robot_namespace)</robotNamespace>
+		<alwaysOn>true</alwaysOn>
+		<updateRate>100</updateRate>
+		<leftJoint>left_mid_wheel</leftJoint>
+		<rightJoint>right_mid_wheel</rightJoint>
+		<wheelSeparation>0.68</wheelSeparation>
+		<wheelDiameter>0.18</wheelDiameter>
+		<torque>20</torque>
+		<commandTopic>/cmd_vel</commandTopic>
+		<odometryTopic>/odom</odometryTopic>
+		<odometryFrame>map</odometryFrame>
+		<robotBaseFrame>base_link</robotBaseFrame>
+		<legacyMode>false</legacyMode>
+		<rosDebugLevel>Debug</rosDebugLevel>
+		<publishWheelTF>true</publishWheelTF>
+		<publishWheelJointState>true</publishWheelJointState>
+		<wheelAcceleration>5</wheelAcceleration>
+		<wheelTorque>20</wheelTorque>
+		<publishTf>1</publishTf>
+		<odometrySource>encoder</odometrySource>
+		</plugin>
+	</gazebo>
+	<gazebo>
 		<plugin name="imu_controller" filename="libhector_gazebo_ros_imu.so">
 			<robotNamespace>$(arg robot_namespace)</robotNamespace>

Commit message: arm updates

File: src/titan_description/urdf/titan.xacro (robot description, xacro)
@@ -18,4 +18,8 @@
 	<xacro:property name="wheel_radius" value="0.09" />
 	<xacro:property name="wheel_length" value="0.0508" />
+	<xacro:property name="computer_x_size" value="0.23"/>
+	<xacro:property name="computer_y_size" value="0.19"/>
+	<xacro:property name="computer_z_size" value="0.11"/>
+	<xacro:property name="computer_mass" value="0.3"/>
 	<xacro:property name="arm_base_x_size" value="0.0381"/>
 	<xacro:property name="arm_base_y_size" value="0.1143"/>
@@ -103,4 +107,7 @@
                 </inertial> -->
         </link>
+	<link name="computer_link">
+		<xacro:make_box x="0.0" y="0.0" z="0.0" roll="0" pitch="0" yaw="0" sizex="${computer_x_size}" sizey="${computer_y_size}" sizez="${computer_z_size}"/>
+	</link>
 	<link name="arm_base_link">
 		<pose xyz="0 0 0" rpy="0 0 0" />
@@ -137,4 +144,9 @@
 		<child link="laser_mount_link"/>
 		<origin xyz="0.31 0.0 0.08" rpy="0 0 0" />
+	</joint>
+	<joint name="base_to_computer" type="fixed">
+		<parent link="base_link"/>
+		<child link="computer_link"/>
+		<origin xyz="${computer_x_size/2 + 0.054} ${-computer_y_size/2} ${computer_z_size/2}" rpy="0 0 0" />
 	</joint>
 	<joint name="base_to_imu_link" type="fixed">

Commit message: arm updates

File: src/titan_description/urdf/titan.xacro (robot description, xacro)
@@ -138,5 +138,5 @@
                 <parent link="base_link"/>
                 <child link="camera_link"/>
-                <origin xyz="0.13 0.08 ${(base_z_size/2) + 0.3}" rpy="0 0 0" />
+                <origin xyz="0.0 0.18 0.6" rpy="0.0 0.55 -0.15" />
         </joint>
 	<joint name="base_to_laser" type="fixed">
