Commit message: updates for camera

File: src/titan_description/urdf/titan.xacro (robot description, xacro)
@@ -34,15 +34,15 @@
 	<xacro:property name="link1_base_z_size" value="0.0381"/>
 	<xacro:property name="link1_base_mass" value="0.05"/>
-	<xacro:property name="link2_base_x_size" value="0.5"/>
+	<xacro:property name="link2_base_x_size" value="0.31"/>
 	<xacro:property name="link2_base_y_size" value="0.0381"/>
 	<xacro:property name="link2_base_z_size" value="0.0381"/>
 	<xacro:property name="link2_base_mass" value="0.05"/>
-	<xacro:property name="link3_base_x_size" value="0.5"/>
+	<xacro:property name="link3_base_x_size" value="0.27"/>
 	<xacro:property name="link3_base_y_size" value="0.0381"/>
 	<xacro:property name="link3_base_z_size" value="0.0381"/>
 	<xacro:property name="link3_base_mass" value="0.05"/>
 	<xacro:property name="eef_x_size" value="0.0381"/>
-	<xacro:property name="eef_y_size" value="0.0381"/>
-	<xacro:property name="eef_z_size" value="0.15"/>
+	<xacro:property name="eef_y_size" value="0.12"/>
+	<xacro:property name="eef_z_size" value="0.10"/>
 	<xacro:property name="eef_mass" value="0.05"/>
 	<xacro:property name="camera_link" value="0.05" />

Commit message: arm updates

File: src/titan_description/urdf/titan.xacro (robot description, xacro)
@@ -175,5 +175,5 @@
 		<parent link="link1"/>
 		<child link="link2"/>
-		<limit effort="1000.0" lower="-2" upper="2" velocity="0.45"/>
+		<limit effort="1000.0" lower="-3" upper="3" velocity="0.40"/>
 		<axis xyz="0 0 1"/>
 		<origin xyz="${link1_base_z_size/2} 0 ${-link1_base_z_size}" rpy="0 0 0" />
@@ -182,5 +182,5 @@
 		<parent link="link2"/>
 		<child link="link3"/>
-		<limit effort="1000.0" lower="-3.0" upper="3.0" velocity="0.255"/>
+		<limit effort="1000.0" lower="-3.0" upper="3.0" velocity="0.40"/>
 		<axis xyz="0 0 1"/>
 		<origin xyz="${link2_base_x_size} 0 ${-link2_base_z_size}" rpy="0 0 0" />
@@ -188,5 +188,5 @@
 	<joint name="link3_to_eef" type="revolute">
 		<parent link="link3"/>
-		<limit effort="1000.0" lower="${-1.57}" upper="1.57" velocity="0.35"/>
+		<limit effort="1000.0" lower="${-1.57}" upper="1.57" velocity="0.40"/>
 		<axis xyz="0 0 1"/>
 		<child link="end_effector"/>

Commit message: arm updates for depth camera

File: src/titan_description/urdf/titan.xacro (robot description, xacro)
@@ -138,5 +138,5 @@
                 <parent link="base_link"/>
                 <child link="camera_link"/>
-                <origin xyz="0.0 0.18 0.6" rpy="0.0 0.55 -0.15" />
+                <origin xyz="0.0 0.15 0.6" rpy="0.0 0.55 -0.15" />
         </joint>
 	<joint name="base_to_laser" type="fixed">

Commit message: teleop updates

File: src/titan_description/urdf/titan.xacro (robot description, xacro)
@@ -138,5 +138,5 @@
                 <parent link="base_link"/>
                 <child link="camera_link"/>
-                <origin xyz="0.0 0.15 0.6" rpy="0.0 0.55 -0.15" />
+                <origin xyz="0.0 0.15 0.6" rpy="0.0 0.63 0.0" />
         </joint>
 	<joint name="base_to_laser" type="fixed">
@@ -165,5 +165,5 @@
 		<limit effort="1000.0" lower="0.0" upper="${arm_base_z_size }" velocity="0.5"/>
 		<axis xyz="0 0 -1"/>
-		<origin xyz="0.05 0 ${arm_base_z_size/2 - zaxis_base_z_size/2}"/>
+		<origin xyz="0.05 0 ${arm_base_z_size/2 - zaxis_base_z_size/2 - 0.0504}"/>
 	</joint>
 	<joint name="zaxis_to_link1" type="fixed">

Commit message: arm stuff

File: src/titan_description/urdf/titan.xacro (robot description, xacro)
@@ -165,5 +165,5 @@
 		<limit effort="1000.0" lower="0.0" upper="${arm_base_z_size }" velocity="0.5"/>
 		<axis xyz="0 0 -1"/>
-		<origin xyz="0.05 0 ${arm_base_z_size/2 - zaxis_base_z_size/2 - 0.0504}"/>
+		<origin xyz="0.05 0 ${arm_base_z_size/2 - zaxis_base_z_size/2 - 0.0254}"/>
 	</joint>
 	<joint name="zaxis_to_link1" type="fixed">

Commit message: titan arm

File: src/titan_description/urdf/titan.xacro (robot description, xacro)
@@ -165,5 +165,5 @@
 		<limit effort="1000.0" lower="0.0" upper="${arm_base_z_size }" velocity="0.5"/>
 		<axis xyz="0 0 -1"/>
-		<origin xyz="0.05 0 ${arm_base_z_size/2 - zaxis_base_z_size/2 - 0.0254}"/>
+		<origin xyz="0.05 0 ${arm_base_z_size/2 - zaxis_base_z_size/2 + 0.0254}"/>
 	</joint>
 	<joint name="zaxis_to_link1" type="fixed">

Commit message: urdf updateS

File: src/titan_description/urdf/titan.xacro (robot description, xacro)
@@ -165,5 +165,5 @@
 		<limit effort="1000.0" lower="0.0" upper="${arm_base_z_size }" velocity="0.5"/>
 		<axis xyz="0 0 -1"/>
-		<origin xyz="0.05 0 ${arm_base_z_size/2 - zaxis_base_z_size/2 + 0.0254}"/>
+		<origin xyz="0.05 0 ${arm_base_z_size/2 - zaxis_base_z_size/2 - 0.075}"/>
 	</joint>
 	<joint name="zaxis_to_link1" type="fixed">

Commit message: arm updates

File: src/titan_description/urdf/titan.xacro (robot description, xacro)
@@ -30,5 +30,5 @@
 	<xacro:property name="zaxis_base_z_size" value="0.1524"/>
 	<xacro:property name="zaxis_base_mass" value="0.05"/>
-	<xacro:property name="link1_base_x_size" value="0.09"/>
+	<xacro:property name="link1_base_x_size" value="0.115"/>
 	<xacro:property name="link1_base_y_size" value="0.0381"/>
 	<xacro:property name="link1_base_z_size" value="0.0381"/>
@@ -138,5 +138,5 @@
                 <parent link="base_link"/>
                 <child link="camera_link"/>
-                <origin xyz="0.0 0.15 0.6" rpy="0.0 0.63 0.0" />
+                <origin xyz="0.025 0.15 0.6" rpy="0.0 0.63 0.0" />
         </joint>
 	<joint name="base_to_laser" type="fixed">
@@ -165,5 +165,5 @@
 		<limit effort="1000.0" lower="0.0" upper="${arm_base_z_size }" velocity="0.5"/>
 		<axis xyz="0 0 -1"/>
-		<origin xyz="0.05 0 ${arm_base_z_size/2 - zaxis_base_z_size/2 - 0.075}"/>
+		<origin xyz="0.09 0 ${arm_base_z_size/2 - zaxis_base_z_size/2 - 0.075}"/>
 	</joint>
 	<joint name="zaxis_to_link1" type="fixed">

Commit message: arm/tray updates

File: src/titan_description/urdf/titan.xacro (robot description, xacro)
@@ -9,4 +9,8 @@
 	<xacro:property name="base_z_size" value="0.0508"/>
 	<xacro:property name="base_mass" value="10"/>
+        <xacro:property name="tray_x_size" value="0.3048"/>
+        <xacro:property name="tray_y_size" value="0.2286"/>
+        <xacro:property name="tray_z_size" value="0.00254"/>
+        <xacro:property name="tray_mass" value="10"/>
 	<xacro:property name="laser_x_size" value="0.125"/>
 	<xacro:property name="laser_y_size" value="0.105"/>
@@ -44,5 +48,5 @@
 	<xacro:property name="eef_x_size" value="0.0381"/>
 	<xacro:property name="eef_y_size" value="0.12"/>
-	<xacro:property name="eef_z_size" value="0.10"/>
+	<xacro:property name="eef_z_size" value="0.08"/>
 	<xacro:property name="eef_mass" value="0.05"/>
 	<xacro:property name="camera_link" value="0.05" />
@@ -110,4 +114,7 @@
 		<xacro:make_box x="0.0" y="0.0" z="0.0" roll="0" pitch="0" yaw="0" sizex="${computer_x_size}" sizey="${computer_y_size}" sizez="${computer_z_size}"/>
 	</link>
+	<link name="tray_link">
+		<xacro:make_box x="0.0" y="0.0" z="0.0" roll="0" pitch="0" yaw="0" sizex="${tray_x_size}" sizey="${tray_y_size}" sizez="${tray_z_size}"/>
+	</link>
 	<link name="arm_base_link">
 		<pose xyz="0 0 0" rpy="0 0 0" />
@@ -150,4 +157,9 @@
 		<origin xyz="${computer_x_size/2 + 0.054} ${-computer_y_size/2} ${computer_z_size/2}" rpy="0 0 0" />
 	</joint>
+	<joint name="base_to_tray" type="fixed">
+		<parent link="base_link"/>
+		<child link="tray_link"/>
+		<origin xyz="${-0.20} ${-0.20} ${tray_z_size/2 + 0.17}" rpy="0 0 0" />
+	</joint>
 	<joint name="base_to_imu_link" type="fixed">
 		<parent link="base_link"/>
@@ -165,10 +177,10 @@
 		<limit effort="1000.0" lower="0.0" upper="${arm_base_z_size }" velocity="0.5"/>
 		<axis xyz="0 0 -1"/>
-		<origin xyz="0.09 0 ${arm_base_z_size/2 - zaxis_base_z_size/2 - 0.075}"/>
+		<origin xyz="0.05 0 ${arm_base_z_size/2 - zaxis_base_z_size/2 - 0.075}"/>
 	</joint>
 	<joint name="zaxis_to_link1" type="fixed">
 		<parent link="zaxis_base_link"/>
 		<child link="link1"/>
-		<origin xyz="${zaxis_base_x_size/2 + link1_base_x_size/2} 0 0" rpy="0 0 0"/>
+		<origin xyz="${zaxis_base_x_size/2 + link1_base_x_size/2 - 0.025} 0 0" rpy="0 0 0"/>
 	</joint>
 	<joint name="link1_to_link2" type="revolute">
@@ -191,5 +203,5 @@
 		<axis xyz="0 0 1"/>
 		<child link="end_effector"/>
-                <origin xyz="${link3_base_x_size} 0 ${-eef_z_size + 0.001}" rpy="0 0 0"/>
+                <origin xyz="${link3_base_x_size} 0 ${-eef_z_size}" rpy="0 0 0"/>
 	</joint>
 	<xacro:titan_wheel wheel_prefix="left_front">

Commit message: FULLY AUTO

File: src/titan_description/urdf/titan.xacro (robot description, xacro)
@@ -30,5 +30,5 @@
 	<xacro:property name="arm_base_z_size" value="0.6096"/>
 	<xacro:property name="arm_base_mass" value="0.3"/>
-	<xacro:property name="zaxis_base_x_size" value="0.0381"/>
+	<xacro:property name="zaxis_base_x_size" value="0.00254"/>
 	<xacro:property name="zaxis_base_y_size" value="0.1143"/>
 	<xacro:property name="zaxis_base_z_size" value="0.1524"/>
@@ -177,22 +177,22 @@
 		<limit effort="1000.0" lower="0.0" upper="${arm_base_z_size }" velocity="0.5"/>
 		<axis xyz="0 0 -1"/>
-		<origin xyz="0.05 0 ${arm_base_z_size/2 - zaxis_base_z_size/2 - 0.075}"/>
+		<origin xyz="0.035 0 ${arm_base_z_size/2 - zaxis_base_z_size/2 - 0.075}"/>
 	</joint>
 	<joint name="zaxis_to_link1" type="fixed">
 		<parent link="zaxis_base_link"/>
 		<child link="link1"/>
-		<origin xyz="${zaxis_base_x_size/2 + link1_base_x_size/2 - 0.025} 0 0" rpy="0 0 0"/>
+		<origin xyz="${zaxis_base_x_size/2 + link1_base_x_size/2} 0 0" rpy="0 0 0"/>
 	</joint>
 	<joint name="link1_to_link2" type="revolute">
 		<parent link="link1"/>
 		<child link="link2"/>
-		<limit effort="1000.0" lower="-3" upper="3" velocity="0.40"/>
+		<limit effort="1000.0" lower="-3.1" upper="3.1" velocity="0.40"/>
 		<axis xyz="0 0 1"/>
-		<origin xyz="${link1_base_z_size/2} 0 ${-link1_base_z_size}" rpy="0 0 0" />
+		<origin xyz="${link1_base_x_size/2} 0 ${-link1_base_z_size}" rpy="0 0 0" />
 	</joint>
 	<joint name="link2_to_link3" type="revolute">
 		<parent link="link2"/>
 		<child link="link3"/>
-		<limit effort="1000.0" lower="-3.0" upper="3.0" velocity="0.40"/>
+		<limit effort="1000.0" lower="-3.1" upper="3.1" velocity="0.40"/>
 		<axis xyz="0 0 1"/>
 		<origin xyz="${link2_base_x_size} 0 ${-link2_base_z_size}" rpy="0 0 0" />
